File: hardware/raspi-aufsatz-v2/raspi-aufsatz-v2.kicad_pcb (KiCad board)
At the start: 2 copper layers, 55.9 x 41.9 mm, 23 parts, among them J1 Raspberry_Pi_2_3, J2 Button, J3 Supply, J4 Screw_Terminal_01x04, J5 Data, J6 USB_A, Q1 IRLZ34N, U1 TXB0104D

Commit message: Hardware raspi-aufsatz-v2 geupdated. Bohrung hinzugefügt und Schraubanschlüsse gedreht.
Parts:
- added REF**: 1pin, Connectors:1pin, F.Cu at (94.5, 94.5)
- moved J4 7.47 mm to (139.7, 70.1), turned to 270 degrees
- moved J2 7.38 mm to (95.8, 87.4), turned to 90 degrees
- moved J5 2.97 mm to (140.0, 82.3), turned to 270 degrees
- moved J3 2.84 mm to (95.8, 73.9), turned to 90 degrees
- moved J6 0.80 mm to (105.7, 85.9)
Routing:
- net Net-(C2-Pad1): track 64.9 -> 36.3 mm
- net Net-(C1-Pad1): track 74.2 -> 55.7 mm, vias 0 -> 2
- net TASTER2: track 55.1 -> 41.2 mm
- net Net-(J2-Pad4): track 42.2 -> 55.1 mm
- net Net-(C3-Pad1): track 48.8 -> 58.0 mm
- net Net-(J5-Pad1): track 15.9 -> 24.1 mm
- net +5VD: track 43.1 -> 49.9 mm
- net Net-(Q1-Pad1): track 41.5 -> 46.5 mm
- net LED: track 34.6 -> 38.5 mm, vias 1 -> 0
- net RGBW_LOW: track 42.6 -> 42.9 mm, vias 1 -> 0
Other:
- board text added: "5 G"
- board text added: "D G"
- board text added: "L- L+ B- B+"
- board text added: "T1 G T2 G"
- board text removed: "B+ B- L+ L-"
- board text removed: "G +5V"
- board text removed: "G D"
- board text removed: "G T2 G T1"
